Commit message: Use osg files for visual meshes in urdf files
  Dae are not displayed correctly in OpenSceneGraph inserted in Qt.

File: ur_description/urdf/ur10.urdf.xacro (robot description, xacro)
@@ -57,5 +57,5 @@
       <visual>
         <geometry>
-          <mesh filename="package://ur_description/meshes/ur10/visual/base.dae"/>
+          <mesh filename="package://ur_description/meshes/ur10/visual/base.osg"/>
         </geometry>
         <material name="LightGrey">
@@ -88,5 +88,5 @@
       <visual>
         <geometry>
-          <mesh filename="package://ur_description/meshes/ur10/visual/shoulder.dae"/>
+          <mesh filename="package://ur_description/meshes/ur10/visual/shoulder.osg"/>
         </geometry>
         <material name="LightGrey">
@@ -119,5 +119,5 @@
       <visual>
         <geometry>
-          <mesh filename="package://ur_description/meshes/ur10/visual/upperarm.dae"/>
+          <mesh filename="package://ur_description/meshes/ur10/visual/upperarm.osg"/>
         </geometry>
         <material name="LightGrey">
@@ -150,5 +150,5 @@
       <visual>
          <geometry>
-          <mesh filename="package://ur_description/meshes/ur10/visual/forearm.dae"/>
+          <mesh filename="package://ur_description/meshes/ur10/visual/forearm.osg"/>
         </geometry>
         <material name="LightGrey">
@@ -181,5 +181,5 @@
       <visual>
         <geometry>
-          <mesh filename="package://ur_description/meshes/ur10/visual/wrist1.dae"/>
+          <mesh filename="package://ur_description/meshes/ur10/visual/wrist1.osg"/>
         </geometry>
         <material name="LightGrey">
@@ -212,5 +212,5 @@
       <visual>
         <geometry>
-          <mesh filename="package://ur_description/meshes/ur10/visual/wrist2.dae"/>
+          <mesh filename="package://ur_description/meshes/ur10/visual/wrist2.osg"/>
         </geometry>
         <material name="LightGrey">
@@ -243,5 +243,5 @@
       <visual>
         <geometry>
-          <mesh filename="package://ur_description/meshes/ur10/visual/wrist3.dae"/>
+          <mesh filename="package://ur_description/meshes/ur10/visual/wrist3.osg"/>
         </geometry>
         <material name="LightGrey">

File: ur_description/urdf/ur3.urdf.xacro (robot description, xacro)
@@ -56,5 +56,5 @@
       <visual>
         <geometry>
-          <mesh filename="package://ur_description/meshes/ur3/visual/base.dae"/>
+          <mesh filename="package://ur_description/meshes/ur3/visual/base.osg"/>
         </geometry>
         <material name="LightGrey">
@@ -87,5 +87,5 @@
       <visual>
         <geometry>
-          <mesh filename="package://ur_description/meshes/ur3/visual/shoulder.dae"/>
+          <mesh filename="package://ur_description/meshes/ur3/visual/shoulder.osg"/>
         </geometry>
         <material name="LightGrey">
@@ -118,5 +118,5 @@
       <visual>
         <geometry>
-          <mesh filename="package://ur_description/meshes/ur3/visual/upperarm.dae"/>
+          <mesh filename="package://ur_description/meshes/ur3/visual/upperarm.osg"/>
         </geometry>
         <material name="LightGrey">
@@ -149,5 +149,5 @@
       <visual>
          <geometry>
-          <mesh filename="package://ur_description/meshes/ur3/visual/forearm.dae"/>
+          <mesh filename="package://ur_description/meshes/ur3/visual/forearm.osg"/>
         </geometry>
         <material name="LightGrey">
@@ -180,5 +180,5 @@
       <visual>
         <geometry>
-          <mesh filename="package://ur_description/meshes/ur3/visual/wrist1.dae"/>
+          <mesh filename="package://ur_description/meshes/ur3/visual/wrist1.osg"/>
         </geometry>
         <material name="LightGrey">
@@ -211,5 +211,5 @@
       <visual>
         <geometry>
-          <mesh filename="package://ur_description/meshes/ur3/visual/wrist2.dae"/>
+          <mesh filename="package://ur_description/meshes/ur3/visual/wrist2.osg"/>
         </geometry>
         <material name="LightGrey">
@@ -242,5 +242,5 @@
       <visual>
         <geometry>
-          <mesh filename="package://ur_description/meshes/ur3/visual/wrist3.dae"/>
+          <mesh filename="package://ur_description/meshes/ur3/visual/wrist3.osg"/>
         </geometry>
         <material name="LightGrey">

File: ur_description/urdf/ur5.urdf.xacro (robot description, xacro)
@@ -72,5 +72,5 @@
       <visual>
         <geometry>
-          <mesh filename="package://ur_description/meshes/ur5/visual/base.dae" />
+          <mesh filename="package://ur_description/meshes/ur5/visual/base.osg" />
         </geometry>
         <material name="LightGrey">
@@ -103,5 +103,5 @@
       <visual>
         <geometry>
-          <mesh filename="package://ur_description/meshes/ur5/visual/shoulder.dae" />
+          <mesh filename="package://ur_description/meshes/ur5/visual/shoulder.osg" />
         </geometry>
         <material name="LightGrey">
@@ -134,5 +134,5 @@
       <visual>
         <geometry>
-          <mesh filename="package://ur_description/meshes/ur5/visual/upperarm.dae" />
+          <mesh filename="package://ur_description/meshes/ur5/visual/upperarm.osg" />
         </geometry>
         <material name="LightGrey">
@@ -165,5 +165,5 @@
       <visual>
         <geometry>
-          <mesh filename="package://ur_description/meshes/ur5/visual/forearm.dae" />
+          <mesh filename="package://ur_description/meshes/ur5/visual/forearm.osg" />
         </geometry>
         <material name="LightGrey">
@@ -196,5 +196,5 @@
       <visual>
         <geometry>
-          <mesh filename="package://ur_description/meshes/ur5/visual/wrist1.dae" />
+          <mesh filename="package://ur_description/meshes/ur5/visual/wrist1.osg" />
         </geometry>
         <material name="LightGrey">
@@ -227,5 +227,5 @@
       <visual>
         <geometry>
-          <mesh filename="package://ur_description/meshes/ur5/visual/wrist2.dae" />
+          <mesh filename="package://ur_description/meshes/ur5/visual/wrist2.osg" />
         </geometry>
         <material name="LightGrey">
@@ -258,5 +258,5 @@
       <visual>
         <geometry>
-          <mesh filename="package://ur_description/meshes/ur5/visual/wrist3.dae" />
+          <mesh filename="package://ur_description/meshes/ur5/visual/wrist3.osg" />
         </geometry>
         <material name="LightGrey">
