Commit message: Move OSG versions of DAE into file.dae.osg instead of file.osg
* The gepetto-viewer finds them automatically so the URDF does not have
* to be modified.

File: ur_description/urdf/ur5.urdf.xacro (robot description, xacro)
@@ -72,5 +72,5 @@
       <visual>
         <geometry>
-          <mesh filename="package://ur_description/meshes/ur5/visual/base.osg" />
+          <mesh filename="package://ur_description/meshes/ur5/visual/base.dae" />
         </geometry>
         <material name="LightGrey">
@@ -103,5 +103,5 @@
       <visual>
         <geometry>
-          <mesh filename="package://ur_description/meshes/ur5/visual/shoulder.osg" />
+          <mesh filename="package://ur_description/meshes/ur5/visual/shoulder.dae" />
         </geometry>
         <material name="LightGrey">
@@ -134,5 +134,5 @@
       <visual>
         <geometry>
-          <mesh filename="package://ur_description/meshes/ur5/visual/upperarm.osg" />
+          <mesh filename="package://ur_description/meshes/ur5/visual/upperarm.dae" />
         </geometry>
         <material name="LightGrey">
@@ -165,5 +165,5 @@
       <visual>
         <geometry>
-          <mesh filename="package://ur_description/meshes/ur5/visual/forearm.osg" />
+          <mesh filename="package://ur_description/meshes/ur5/visual/forearm.dae" />
         </geometry>
         <material name="LightGrey">
@@ -196,5 +196,5 @@
       <visual>
         <geometry>
-          <mesh filename="package://ur_description/meshes/ur5/visual/wrist1.osg" />
+          <mesh filename="package://ur_description/meshes/ur5/visual/wrist1.dae" />
         </geometry>
         <material name="LightGrey">
@@ -227,5 +227,5 @@
       <visual>
         <geometry>
-          <mesh filename="package://ur_description/meshes/ur5/visual/wrist2.osg" />
+          <mesh filename="package://ur_description/meshes/ur5/visual/wrist2.dae" />
         </geometry>
         <material name="LightGrey">
@@ -258,5 +258,5 @@
       <visual>
         <geometry>
-          <mesh filename="package://ur_description/meshes/ur5/visual/wrist3.osg" />
+          <mesh filename="package://ur_description/meshes/ur5/visual/wrist3.dae" />
         </geometry>
         <material name="LightGrey">
